File: Set-up ensayo/Set-up ensayo.sch (KiCad schematic (older format))
At the start: 17 parts, among them J1 Conn_Coaxial, J2 DB9_Female_MountingHoles

Commit message: Cambié los footprints en el archivo .net y en el esquemático
Parts:
- JP1, JP2: footprint Footprints proyecto:PinHeader_1x02_P1.00mm_Vertical -> Footprints proyecto:PinHeader_1x02_P2.54mm_Vertical
- TP1, TP2, TP3, TP4, TP5, TP6: footprint Footprints proyecto:PinHeader_1x01_P1.00mm_Horizontal -> Footprints proyecto:PinHeader_1x01_P2.54mm_Horizontal
Changed lines of the file:
@@
 F 0 "TP3" H 3903 3401 50  0000 L CNN
 F 1 "TestPoint_Probe" H 3903 3310 50  0000 L CNN
-F 2 "Footprints proyecto:PinHeader_1x01_P1.00mm_Horizontal" H 3950 3300 50  0001 C CNN
+F 2 "Footprints proyecto:PinHeader_1x01_P2.54mm_Horizontal" H 3950 3300 50  0001 C CNN
 F 3 "~" H 3950 3300 50  0001 C CNN
 F 4 "Interfaz eléctrica con punta de medición V1 osciloscopio" H 3750 3300 50  0001 C CNN "Función"
@@
 F 0 "TP5" H 6703 3351 50  0000 L CNN
 F 1 "TestPoint_Probe" H 6703 3260 50  0000 L CNN
-F 2 "Footprints proyecto:PinHeader_1x01_P1.00mm_Horizontal" H 6750 3250 50  0001 C CNN
+F 2 "Footprints proyecto:PinHeader_1x01_P2.54mm_Horizontal" H 6750 3250 50  0001 C CNN
 F 3 "~" H 6750 3250 50  0001 C CNN
 F 4 "Interfaz eléctrica con punta de medición V2 osciloscopio" H 6550 3250 50  0001 C CNN "Función"
@@
 F 0 "TP6" H 6658 4318 50  0000 L CNN
 F 1 "TestPoint" H 6658 4227 50  0000 L CNN
-F 2 "Footprints proyecto:PinHeader_1x01_P1.00mm_Horizontal" H 6800 4200 50  0001 C CNN
+F 2 "Footprints proyecto:PinHeader_1x01_P2.54mm_Horizontal" H 6800 4200 50  0001 C CNN
 F 3 "~" H 6800 4200 50  0001 C CNN
 F 4 "Interfaz eléctrica con GND de V2 osciloscopio" H 6600 4200 50  0001 C CNN "Función"
@@
 F 0 "TP4" H 3758 4318 50  0000 L CNN
 F 1 "TestPoint" H 3758 4227 50  0000 L CNN
-F 2 "Footprints proyecto:PinHeader_1x01_P1.00mm_Horizontal" H 3900 4200 50  0001 C CNN
+F 2 "Footprints proyecto:PinHeader_1x01_P2.54mm_Horizontal" H 3900 4200 50  0001 C CNN
 F 3 "~" H 3900 4200 50  0001 C CNN
 F 4 "Interfaz eléctrica con GND de V1 osciloscopio" H 3700 4200 50  0001 C CNN "Función"
@@
 F 0 "TP1" H 2958 3418 50  0000 L CNN
 F 1 "TestPoint_Alt" H 2958 3327 50  0000 L CNN
-F 2 "Footprints proyecto:PinHeader_1x01_P1.00mm_Horizontal" H 3100 3300 50  0001 C CNN
+F 2 "Footprints proyecto:PinHeader_1x01_P2.54mm_Horizontal" H 3100 3300 50  0001 C CNN
 F 3 "~" H 3100 3300 50  0001 C CNN
 F 4 "Interfaz eléctrica con potencial positivo tester" H 2900 3300 50  0001 C CNN "Función"
@@
 F 0 "TP2" H 2908 4318 50  0000 L CNN
 F 1 "TestPoint" H 2908 4227 50  0000 L CNN
-F 2 "Footprints proyecto:PinHeader_1x01_P1.00mm_Horizontal" H 3050 4200 50  0001 C CNN
+F 2 "Footprints proyecto:PinHeader_1x01_P2.54mm_Horizontal" H 3050 4200 50  0001 C CNN
 F 3 "~" H 3050 4200 50  0001 C CNN
 F 4 "Interfaz eléctrica con potencial negativo tester" H 2850 4200 50  0001 C CNN "Función"
@@
 F 0 "JP1" H 5700 3612 50  0000 C CNN
 F 1 "Jumper_NC_Small" H 5700 3521 50  0000 C CNN
-F 2 "Footprints proyecto:PinHeader_1x02_P1.00mm_Vertical" H 5700 3400 50  0001 C CNN
+F 2 "Footprints proyecto:PinHeader_1x02_P2.54mm_Vertical" H 5700 3400 50  0001 C CNN
 F 3 "~" H 5700 3400 50  0001 C CNN
 F 4 "Jumper para configuración de resistencia fija" H 5700 3400 50  0001 C CNN "Función"
@@
 F 0 "JP2" H 5700 3935 50  0000 C CNN
 F 1 "Jumper_NO_Small" H 5700 3844 50  0000 C CNN
-F 2 "Footprints proyecto:PinHeader_1x02_P1.00mm_Vertical" H 5700 3750 50  0001 C CNN
+F 2 "Footprints proyecto:PinHeader_1x02_P2.54mm_Vertical" H 5700 3750 50  0001 C CNN
 F 3 "~" H 5700 3750 50  0001 C CNN
 F 4 "Jumper para configuración de resistencia variable" H 5700 3750 50  0001 C CNN "Función"

Commit message: Cambio de footprint horizontal por verticales para pines de medicion y ruteo de las pistas correspondientes
Parts:
- TP1, TP2, TP3, TP4, TP5, TP6: footprint Footprints proyecto:PinHeader_1x01_P2.54mm_Horizontal -> Footprints proyecto:PinHeader_1x01_P2.54mm_Vertical
Changed lines of the file:
@@
 F 0 "TP3" H 3903 3401 50  0000 L CNN
 F 1 "TestPoint_Probe" H 3903 3310 50  0000 L CNN
-F 2 "Footprints proyecto:PinHeader_1x01_P2.54mm_Horizontal" H 3950 3300 50  0001 C CNN
+F 2 "Footprints proyecto:PinHeader_1x01_P2.54mm_Vertical" H 3950 3300 50  0001 C CNN
 F 3 "~" H 3950 3300 50  0001 C CNN
 F 4 "Interfaz eléctrica con punta de medición V1 osciloscopio" H 3750 3300 50  0001 C CNN "Función"
@@
 F 0 "TP5" H 6703 3351 50  0000 L CNN
 F 1 "TestPoint_Probe" H 6703 3260 50  0000 L CNN
-F 2 "Footprints proyecto:PinHeader_1x01_P2.54mm_Horizontal" H 6750 3250 50  0001 C CNN
+F 2 "Footprints proyecto:PinHeader_1x01_P2.54mm_Vertical" H 6750 3250 50  0001 C CNN
 F 3 "~" H 6750 3250 50  0001 C CNN
 F 4 "Interfaz eléctrica con punta de medición V2 osciloscopio" H 6550 3250 50  0001 C CNN "Función"
@@
 F 0 "TP6" H 6658 4318 50  0000 L CNN
 F 1 "TestPoint" H 6658 4227 50  0000 L CNN
-F 2 "Footprints proyecto:PinHeader_1x01_P2.54mm_Horizontal" H 6800 4200 50  0001 C CNN
+F 2 "Footprints proyecto:PinHeader_1x01_P2.54mm_Vertical" H 6800 4200 50  0001 C CNN
 F 3 "~" H 6800 4200 50  0001 C CNN
 F 4 "Interfaz eléctrica con GND de V2 osciloscopio" H 6600 4200 50  0001 C CNN "Función"
@@
 F 0 "TP4" H 3758 4318 50  0000 L CNN
 F 1 "TestPoint" H 3758 4227 50  0000 L CNN
-F 2 "Footprints proyecto:PinHeader_1x01_P2.54mm_Horizontal" H 3900 4200 50  0001 C CNN
+F 2 "Footprints proyecto:PinHeader_1x01_P2.54mm_Vertical" H 3900 4200 50  0001 C CNN
 F 3 "~" H 3900 4200 50  0001 C CNN
 F 4 "Interfaz eléctrica con GND de V1 osciloscopio" H 3700 4200 50  0001 C CNN "Función"
@@
 F 0 "TP1" H 2958 3418 50  0000 L CNN
 F 1 "TestPoint_Alt" H 2958 3327 50  0000 L CNN
-F 2 "Footprints proyecto:PinHeader_1x01_P2.54mm_Horizontal" H 3100 3300 50  0001 C CNN
+F 2 "Footprints proyecto:PinHeader_1x01_P2.54mm_Vertical" H 3100 3300 50  0001 C CNN
 F 3 "~" H 3100 3300 50  0001 C CNN
 F 4 "Interfaz eléctrica con potencial positivo tester" H 2900 3300 50  0001 C CNN "Función"
@@
 F 0 "TP2" H 2908 4318 50  0000 L CNN
 F 1 "TestPoint" H 2908 4227 50  0000 L CNN
-F 2 "Footprints proyecto:PinHeader_1x01_P2.54mm_Horizontal" H 3050 4200 50  0001 C CNN
+F 2 "Footprints proyecto:PinHeader_1x01_P2.54mm_Vertical" H 3050 4200 50  0001 C CNN
 F 3 "~" H 3050 4200 50  0001 C CNN
 F 4 "Interfaz eléctrica con potencial negativo tester" H 2850 4200 50  0001 C CNN "Función"
