File: Set-up ensayo/Footprints.kicad_pcb (KiCad board)
At the start: 2 copper layers, 114.3 x 63.5 mm, 14 parts, among them J1 Conn_Coaxial, J2 DB9_Female_MountingHoles

Commit message: Actualizción de archivos de footprints
Parts:
- added JP1: Jumper_NC_Small, Footprints proyecto:PinHeader_1x02_P2.54mm_Vertical, F.Cu at (158.1, 83.8)
- added JP2: Jumper_NO_Small, Footprints proyecto:PinHeader_1x02_P2.54mm_Vertical, F.Cu at (170.2, 83.8)
- added RV1: R_POT, Footprints proyecto:Potentiometer_Vishay_248GJ-249GJ_Single_Vertical, F.Cu at (135.3, 92.1)
- H1, H2, H3, H4: footprint MountingHole:MountingHole_2.2mm_M2_ISO7380_Pad -> Footprints proyecto:MountingHole_3.2mm_M3_ISO14580_Pad
- J1: footprint Connector_Coaxial:BNC_TEConnectivity_1478204_Vertical -> Footprints proyecto:BNC_TEConnectivity_1478204_Vertical
- J2: footprint Connector_Dsub:DSUB-9_Female_Horizontal_P2.77x2.84mm_EdgePinOffset4.94mm_Housed_MountingHolesOffset7.48mm -> Footprints proyecto:DSUB-9_Female_Horizontal_P2.77x2.84mm_EdgePinOffset4.94mm_Housed_MountingHolesOffset7.48mm
- MCB1: footprint digikey-footprints:Switch_Toggle_ATE1D-2M3-10-Z -> Footprints proyecto:Switch_Toggle_ATE1D-2M3-10-Z
- R1: footprint Resistor_THT:R_Axial_DIN0204_L3.6mm_D1.6mm_P5.08mm_Horizontal -> Footprints proyecto:R_Axial_DIN0204_L3.6mm_D1.6mm_P7.62mm_Horizontal
- TP1, TP2, TP3, TP4, TP5, TP6: footprint Connector_PinHeader_1.00mm:PinHeader_1x01_P1.00mm_Horizontal -> Footprints proyecto:PinHeader_1x01_P2.54mm_Vertical
- moved H2 63.8 mm to (118.1, 132.1)
- moved MCB1 62.2 mm to (101.6, 121.9)
- moved TP1 48.9 mm to (179.7, 94.0)
- moved TP6 47.2 mm to (179.7, 127.0)
- moved H1 37.9 mm to (132.7, 132.1)
- moved H4 36.9 mm to (161.3, 132.1)
- moved TP2 35.9 mm to (179.7, 101.0)
- moved TP4 35.7 mm to (179.7, 114.3)
- moved TP5 35.3 mm to (179.7, 120.7)
- moved TP3 35.2 mm to (179.7, 107.3)
- moved H3 33.9 mm to (146.7, 132.1)
- moved R1 33.2 mm to (132.9, 119.1)
- moved J1 23.4 mm to (161.3, 100.3)
- moved J2 10.5 mm to (116.2, 94.6)
Connections:
- R1 pad 1: /Vi -> Net-(JP1-Pad2)
Other:
- board text added: "Placa para probar footprints Fecha: 20/08/2019 Autor: Gustavo V. Diaz"
- board text removed: "Placa para probar footprints Fecha: 08/08/2019 Autor: Gustavo V. Diaz"
