File: Set-up ensayo/Set-up ensayo.kicad_pcb (KiCad board)
At the start: 2 copper layers, 53.3 x 61 mm, 17 parts, among them J1 Conn_Coaxial, J2 DB9_Female_MountingHoles

Commit message: Finalicé 6to paso de proceso de diseño de PCB
Parts:
- added REF**: KiCad-Logo2_5mm_SilkScreen, Symbol:KiCad-Logo2_5mm_SilkScreen, F.Cu at (104.8, 92.7)
Other:
- board text added: "Autor: Gustavo V. Diaz Proyecto: PCB ensayo estático Versión: V0.1 Contacto: gus838@gmail.com BS AS - 2019"
- board text added: "JP1: R1 JP2: RV1"
- board text added: "MODO PCB: Ensayo/Ajuste"
- board text added: "Osc. V1"
- board text added: "Osc. V2"
- board text added: "Tester"

Commit message: Finalicé 7mo paso de proceso de diseño de PCB
Other:
- board text added: "+ Osc. V1 -"
- board text added: "+ Osc. V2 -"
- board text added: "+ Tester -"
- board text removed: "Osc. V1"
- board text removed: "Osc. V2"
- board text removed: "Tester"
Changed lines of the file:
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@@
     (effects (font (size 1 1) (thickness 0.15)) (justify left))
   )
-  (gr_text "Osc. V2" (at 139.065 127.635) (layer F.SilkS)
+  (gr_text "+ Osc. V2 -" (at 139.065 133.985) (layer F.SilkS)
     (effects (font (size 1 1) (thickness 0.15)))
   )
-  (gr_text "Osc. V1" (at 127 127.635) (layer F.SilkS)
+  (gr_text "+ Osc. V1 -" (at 128.905 133.985) (layer F.SilkS)
     (effects (font (size 1 1) (thickness 0.15)) (justify right))
   )
-  (gr_text Tester (at 111.125 127.635) (layer F.SilkS)
+  (gr_text "+ Tester -" (at 113.03 133.985) (layer F.SilkS)
     (effects (font (size 1 1) (thickness 0.15)) (justify right))
   )
